File: Untitled.kicad_pcb (KiCad board)
At the start: 2 copper layers, 48.8 x 56.3 mm, 18 parts, among them IC1 MJE340G, U1 LR8N3-G

Commit message: Cap added
Parts:
- C1: footprint MountingHole:MountingHole_2.2mm_M2_DIN965_Pad -> Capacitor_THT:C_Disc_D6.0mm_W2.5mm_P5.00mm
- R3: value R -> 330
- moved C1 0.54 mm to (129.7, 107.9)
Changed lines of the file:
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@@
       (effects (font (size 1 1) (thickness 0.15)))
     )
-    (fp_text value "R" (at 3.81 1.92) (layer "F.Fab")
+    (fp_text value "330" (at 3.81 1.92) (layer "F.Fab")
       (effects (font (size 1 1) (thickness 0.15)))
     )
@@
     )
     (fp_line (start 6.19 1.195) (end 6.19 -1.805) (layer "F.SilkS") (width 0.2))
+    (fp_line (start -1.61 -1.805) (end -1.61 0) (layer "F.SilkS") (width 0.2))
     (fp_line (start 6.19 -1.805) (end -1.61 -1.805) (layer "F.SilkS") (width 0.2))
-    (fp_line (start -1.61 -1.805) (end -1.61 0) (layer "F.SilkS") (width 0.2))
-    (fp_line (start -1.86 -2.055) (end 6.44 -2.055) (layer "F.CrtYd") (width 0.05))
     (fp_line (start -1.86 1.445) (end -1.86 -2.055) (layer "F.CrtYd") (width 0.05))
     (fp_line (start 6.44 -2.055) (end 6.44 1.445) (layer "F.CrtYd") (width 0.05))
+    (fp_line (start -1.86 -2.055) (end 6.44 -2.055) (layer "F.CrtYd") (width 0.05))
     (fp_line (start 6.44 1.445) (end -1.86 1.445) (layer "F.CrtYd") (width 0.05))
+    (fp_line (start -1.61 -1.805) (end 6.19 -1.805) (layer "F.Fab") (width 0.1))
+    (fp_line (start 6.19 1.195) (end -1.61 1.195) (layer "F.Fab") (width 0.1))
     (fp_line (start -1.61 1.195) (end -1.61 -1.805) (layer "F.Fab") (width 0.1))
     (fp_line (start 6.19 -1.805) (end 6.19 1.195) (layer "F.Fab") (width 0.1))
-    (fp_line (start -1.61 -1.805) (end 6.19 -1.805) (layer "F.Fab") (width 0.1))
     (fp_line (start -1.61 -0.66) (end -0.465 -1.805) (layer "F.Fab") (width 0.1))
-    (fp_line (start 6.19 1.195) (end -1.61 1.195) (layer "F.Fab") (width 0.1))
     (pad "1" thru_hole rect locked (at 0 0) (size 1.95 1.95) (drill 1.3) (layers *.Cu *.Mask)
       (net 5 "Net-(C1-Pad1)") (pinfunction "EMITTER") (pintype "passive"))
@@
     )
   )
+  (footprint "Capacitor_THT:C_Disc_D6.0mm_W2.5mm_P5.00mm" (layer "F.Cu")
+    (at 129.725 107.875 180)
+    (descr "C, Disc series, Radial, pin pitch=5.00mm, , diameter*width=6*2.5mm^2, Capacitor, http://cdn-reichelt.de/documents/datenblatt/B300/DS_KERKO_TC.pdf")
+    (tags "C Disc series Radial pin pitch 5.00mm  diameter 6mm width 2.5mm Capacitor")
+    (property "Sheetfile" "Untitled.kicad_sch")
+    (property "Sheetname" "")
+    (attr through_hole)
+    (fp_text reference "C1" (at 2.5 -2.5 180) (layer "F.SilkS")
+      (effects (font (size 1 1) (thickness 0.15)))
+    )
+    (fp_text value "100n" (at 2.5 2.5 180) (layer "F.Fab")
+      (effects (font (size 1 1) (thickness 0.15)))
+    )
+    (fp_text user "${REFERENCE}" (at 2.5 0 180) (layer "F.Fab")
+      (effects (font (size 1 1) (thickness 0.15)))
+    )
+    (fp_line (start -0.62 -1.37) (end -0.62 -0.925) (layer "F.SilkS") (width 0.12))
+    (fp_line (start -0.62 1.37) (end 5.62 1.37) (layer "F.SilkS") (width 0.12))
+    (fp_line (start 5.62 0.925) (end 5.62 1.37) (layer "F.SilkS") (width 0.12))
+    (fp_line (start -0.62 -1.37) (end 5.62 -1.37) (layer "F.SilkS") (width 0.12))
+    (fp_line (start -0.62 0.925) (end -0.62 1.37) (layer "F.SilkS") (width 0.12))
+    (fp_line (start 5.62 -1.37) (end 5.62 -0.925) (layer "F.SilkS") (width 0.12))
+    (fp_line (start -1.05 1.5) (end 6.05 1.5) (layer "F.CrtYd") (width 0.05))
+    (fp_line (start 6.05 1.5) (end 6.05 -1.5) (layer "F.CrtYd") (width 0.05))
+    (fp_line (start -1.05 -1.5) (end -1.05 1.5) (layer "F.CrtYd") (width 0.05))
+    (fp_line (start 6.05 -1.5) (end -1.05 -1.5) (layer "F.CrtYd") (width 0.05))
+    (fp_line (start 5.5 -1.25) (end -0.5 -1.25) (layer "F.Fab") (width 0.1))
+    (fp_line (start -0.5 1.25) (end 5.5 1.25) (layer "F.Fab") (width 0.1))
+    (fp_line (start -0.5 -1.25) (end -0.5 1.25) (layer "F.Fab") (width 0.1))
+    (fp_line (start 5.5 1.25) (end 5.5 -1.25) (layer "F.Fab") (width 0.1))
+    (pad "1" thru_hole circle (at 0 0 180) (size 1.6 1.6) (drill 0.8) (layers *.Cu *.Mask)
+      (net 5 "Net-(C1-Pad1)") (pintype "passive"))
+    (pad "2" thru_hole circle (at 5 0 180) (size 1.6 1.6) (drill 0.8) (layers *.Cu *.Mask)
+      (net 1 "GND") (pintype "passive"))
+    (model "${KICAD6_3DMODEL_DIR}/Capacitor_THT.3dshapes/C_Disc_D6.0mm_W2.5mm_P5.00mm.wrl"
+      (offset (xyz 0 0 0))
+      (scale (xyz 1 1 1))
+      (rotate (xyz 0 0 0))
+    )
+  )
   (footprint "MountingHole:MountingHole_2.2mm_M2_DIN965_Pad" (layer "F.Cu")
-    (at 129.6 107.35 180)
-    (descr "Mounting Hole 2.2mm, M2, DIN965")
-    (tags "mounting hole 2.2mm m2 din965")
-    (property "Sheetfile" "Untitled.kicad_sch")
-    (property "Sheetname" "")
-    (attr exclude_from_pos_files)
-    (fp_text reference "C1" (at 0 -2.9 180) (layer "F.SilkS")
-      (effects (font (size 1 1) (thickness 0.15)))
-    )
-    (fp_text value "100n" (at 0 2.9 180) (layer "F.Fab")
-      (effects (font (size 1 1) (thickness 0.15)))
-    )
-    (fp_text user "${REFERENCE}" (at 0 0 180) (layer "F.Fab")
-      (effects (font (size 1 1) (thickness 0.15)))
-    )
-    (fp_circle (center 0 0) (end 1.9 0) (layer "Cmts.User") (width 0.15) (fill none))
-    (fp_circle (center 0 0) (end 2.15 0) (layer "F.CrtYd") (width 0.05) (fill none))
-    (pad "1" thru_hole circle (at 0 0 180) (size 3.8 3.8) (drill 2.2) (layers *.Cu *.Mask)
-      (net 5 "Net-(C1-Pad1)") (pintype "passive"))
-  )
-  (footprint "MountingHole:MountingHole_2.2mm_M2_DIN965_Pad" (layer "F.Cu")
