File: Untitled.kicad_sch (KiCad schematic)
At the start: 18 parts, among them IC1 MJE340G, U1 LR8N3-G

Commit message: Cap added
Parts:
- C1: footprint MountingHole:MountingHole_2.2mm_M2_DIN965_Pad -> Capacitor_THT:C_Disc_D6.0mm_W2.5mm_P5.00mm
Changed lines of the file:
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@@
       (effects (font (size 1.27 1.27)) (justify left))
     )
-    (property "Footprint" "MountingHole:MountingHole_2.2mm_M2_DIN965_Pad" (id 2) (at 107.6452 95.25 0)
+    (property "Footprint" "Capacitor_THT:C_Disc_D6.0mm_W2.5mm_P5.00mm" (id 2) (at 107.6452 95.25 0)
       (effects (font (size 1.27 1.27)) hide)
     )
@@
     )
     (path "/566517f2-959a-4b71-80c3-b27c8262c664"
-      (reference "C1") (unit 1) (value "100n") (footprint "MountingHole:MountingHole_2.2mm_M2_DIN965_Pad")
+      (reference "C1") (unit 1) (value "100n") (footprint "Capacitor_THT:C_Disc_D6.0mm_W2.5mm_P5.00mm")
     )
     (path "/2d2eced5-bd5f-418b-9cda-232e5080fe2b"
